Commit message: steady go1 training

File: legged_gym/resources/robots/go1/urdf/go1.urdf (robot description, URDF)
Before this commit: robot go1_description, 38 links, 37 joints
Links:
- link FL_calf: geometry collision box size=0.213 0.016 0.016; visual mesh filename=/home/sdalal/project_test/extreme-parkour/legged_gym/resour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 scale=1 1 1
- link FL_hip: geometry visual mesh filename=/home/sdalal/project_test/extreme-parkour/legged_gym/resour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 scale=1 1 1
- link FL_thigh: geometry collision box size=0.213 0.0245 0.034; visual mesh filename=/home/sdalal/project_test/extreme-parkour/legged_gym/resour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 scale=1 1 1
- link FR_calf: geometry collision box size=0.213 0.016 0.016; visual mesh filename=/home/sdalal/project_test/extreme-parkour/legged_gym/resour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 scale=1 1 1
- link FR_hip: geometry visual mesh filename=/home/sdalal/project_test/extreme-parkour/legged_gym/resour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 scale=1 1 1
- link FR_thigh: geometry collision box size=0.213 0.0245 0.034; visual mesh filename=/home/sdalal/project_test/extreme-parkour/legged_gym/resour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 scale=1 1 1
- link RL_calf: geometry collision box size=0.213 0.016 0.016; visual mesh filename=/home/sdalal/project_test/extreme-parkour/legged_gym/resour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 scale=1 1 1
- link RL_hip: geometry visual mesh filename=/home/sdalal/project_test/extreme-parkour/legged_gym/resour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 scale=1 1 1
- link RL_thigh: geometry collision box size=0.213 0.0245 0.034; visual mesh filename=/home/sdalal/project_test/extreme-parkour/legged_gym/resour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 scale=1 1 1
- link RR_calf: geometry collision box size=0.213 0.016 0.016; visual mesh filename=/home/sdalal/project_test/extreme-parkour/legged_gym/resour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 scale=1 1 1
- link RR_hip: geometry visual mesh filename=/home/sdalal/project_test/extreme-parkour/legged_gym/resour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 scale=1 1 1
- link RR_thigh: geometry collision box size=0.213 0.0245 0.034; visual mesh filename=/home/sdalal/project_test/extreme-parkour/legged_gym/resour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 scale=1 1 1
- link camera_chin: geometry collision box size=.001 .001 .001; visual mesh filename=/home/sdalal/project_test/extreme-parkour/legged_gym/resour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 scale=1 1 1
- link camera_face: geometry collision box size=.001 .001 .001; visual mesh filename=/home/sdalal/project_test/extreme-parkour/legged_gym/resour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 scale=1 1 1
- link camera_left: geometry collision box size=.001 .001 .001; visual mesh filename=/home/sdalal/project_test/extreme-parkour/legged_gym/resour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 scale=1 1 1
- link camera_rearDown: geometry collision box size=.001 .001 .001; visual mesh filename=/home/sdalal/project_test/extreme-parkour/legged_gym/resour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 scale=1 1 1
- link camera_right: geometry collision box size=.001 .001 .001; visual mesh filename=/home/sdalal/project_test/extreme-parkour/legged_gym/resour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 scale=1 1 1
- link trunk: geometry collision box size=0.45 0.0935 0.114; visual mesh filename=/home/sdalal/project_test/extreme-parkour/legged_gym/resour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 scale=1 1 1
- link ultraSound_face: geometry collision box size=.001 .001 .001; visual mesh filename=/home/sdalal/project_test/extreme-parkour/legged_gym/resour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 scale=1 1 1
- link ultraSound_left: geometry collision box size=.001 .001 .001; visual mesh filename=/home/sdalal/project_test/extreme-parkour/legged_gym/resour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 scale=1 1 1
- link ultraSound_right: geometry collision box size=.001 .001 .001; visual mesh filename=/home/sdalal/project_test/extreme-parkour/legged_gym/resour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 scale=1 1 1

Commit message: collision boundry change

File: legged_gym/resources/robots/go1/urdf/go1.urdf (robot description, URDF)
Before this commit: robot go1_description, 38 links, 37 joints
Links:
- link FL_calf: geometry collision box size=0.213 0.016 0.016; visual mesh filename=file:///home/sdalal/ws/winter_project/src/isaacgym/docker/e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 scale=1 1 1
- link FL_hip: geometry visual mesh filename=file:///home/sdalal/ws/winter_project/src/isaacgym/docker/e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 scale=1 1 1
- link FL_thigh: geometry collision box size=0.213 0.0245 0.034; visual mesh filename=file:///home/sdalal/ws/winter_project/src/isaacgym/docker/e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 scale=1 1 1
- link FR_calf: geometry collision box size=0.213 0.016 0.016; visual mesh filename=file:///home/sdalal/ws/winter_project/src/isaacgym/docker/e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 scale=1 1 1
- link FR_hip: geometry visual mesh filename=file:///home/sdalal/ws/winter_project/src/isaacgym/docker/e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 scale=1 1 1
- link FR_thigh: geometry collision box size=0.213 0.0245 0.034; visual mesh filename=file:///home/sdalal/ws/winter_project/src/isaacgym/docker/e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 scale=1 1 1
- link RL_calf: geometry collision box size=0.213 0.016 0.016; visual mesh filename=file:///home/sdalal/ws/winter_project/src/isaacgym/docker/e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 scale=1 1 1
- link RL_hip: geometry visual mesh filename=file:///home/sdalal/ws/winter_project/src/isaacgym/docker/e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 scale=1 1 1
- link RL_thigh: geometry collision box size=0.213 0.0245 0.034; visual mesh filename=file:///home/sdalal/ws/winter_project/src/isaacgym/docker/e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 scale=1 1 1
- link RR_calf: geometry collision box size=0.213 0.016 0.016; visual mesh filename=file:///home/sdalal/ws/winter_project/src/isaacgym/docker/e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 scale=1 1 1
- link RR_hip: geometry visual mesh filename=file:///home/sdalal/ws/winter_project/src/isaacgym/docker/e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 scale=1 1 1
- link RR_thigh: geometry collision box size=0.213 0.0245 0.034; visual mesh filename=file:///home/sdalal/ws/winter_project/src/isaacgym/docker/e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 scale=1 1 1
- link camera_chin: geometry collision box size=.001 .001 .001; visual mesh filename=file:///home/sdalal/ws/winter_project/src/isaacgym/docker/e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 scale=1 1 1
- link camera_face: geometry collision box size=.001 .001 .001; visual mesh filename=file:///home/sdalal/ws/winter_project/src/isaacgym/docker/e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 scale=1 1 1
- link camera_left: geometry collision box size=.001 .001 .001; visual mesh filename=file:///home/sdalal/ws/winter_project/src/isaacgym/docker/e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 scale=1 1 1
- link camera_rearDown: geometry collision box size=.001 .001 .001; visual mesh filename=file:///home/sdalal/ws/winter_project/src/isaacgym/docker/e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 scale=1 1 1
- link camera_right: geometry collision box size=.001 .001 .001; visual mesh filename=file:///home/sdalal/ws/winter_project/src/isaacgym/docker/e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 scale=1 1 1
- link trunk: geometry collision box size=0.45 0.0935 0.114; visual mesh filename=file:///home/sdalal/ws/winter_project/src/isaacgym/docker/e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 scale=1 1 1
- link ultraSound_face: geometry collision box size=.001 .001 .001; visual mesh filename=file:///home/sdalal/ws/winter_project/src/isaacgym/docker/e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 scale=1 1 1
- link ultraSound_left: geometry collision box size=.001 .001 .001; visual mesh filename=file:///home/sdalal/ws/winter_project/src/isaacgym/docker/e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 scale=1 1 1
- link ultraSound_right: geometry collision box size=.001 .001 .001; visual mesh filename=file:///home/sdalal/ws/winter_project/src/isaacgym/docker/e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 scale=1 1 1

File: legged_gym/resources/robots/go1/urdf/go1_new.urdf (robot description, URDF)
Before this commit: robot go1_description, 38 links, 37 joints
Links:
- link trunk: geometry collision box size=0.50 0.1935 0.05; visual mesh filename=../meshes/trunk.dae scale=1 1 1
